File: hardware/base.kicad_sch (KiCad schematic)
At the start: 4 parts, among them J1 USB_C_Receptacle_USB2.0_14P, J2 FFC2B21-40-T_REVA, U1 BQ21040DBVR

Commit message: updates
Parts:
- removed J2: FFC2B21-40-T_REVA, footprints:GCT_FFC2B21-40-T_REVA, symbol FFC2B21-40-T_REVA:FFC2B21-40-T_REVA
Other:
- added sheet MODULE_BUS (MODULE_BUS.kicad_sch)
Changed lines of the file:
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@@
 		)
 	)
-	(symbol
-		(lib_id "FFC2B21-40-T_REVA:FFC2B21-40-T_REVA")
-		(at 222.25 72.39 0)
-		(unit 1)
-		(exclude_from_sim no)
-		(in_bom yes)
-		(on_board yes)
-		(dnp no)
+	(sheet
+		(at 54.61 80.01)
+		(size 31.75 31.75)
 		(fields_autoplaced yes)
-		(property "Reference" "J2"
-			(at 229.108 73.66 0)
+		(stroke
+			(width 0.1524)
+			(type solid)
+		)
+		(fill
+			(color 0 0 0 0.0000)
+		)
+		(property "Sheetname" "MODULE_BUS"
+			(at 54.61 79.2984 0)
 			(effects
 				(font
 					(size 1.27 1.27)
 				)
-				(justify left)
+				(justify left bottom)
 			)
 		)
-		(property "Value" "FFC2B21-40-T_REVA"
-			(at 229.108 76.2 0)
+		(property "Sheetfile" "MODULE_BUS.kicad_sch"
+			(at 54.61 112.3446 0)
 			(effects
 				(font
 					(size 1.27 1.27)
 				)
-				(justify left)
+				(justify left top)
 			)
-		)
-		(property "Footprint" "footprints:GCT_FFC2B21-40-T_REVA"
-			(at 222.25 72.39 0)
-			(effects
-				(font
-					(size 1.27 1.27)
-				)
-				(justify bottom)
-				(hide yes)
-			)
-		)
-		(property "Datasheet" ""
-			(at 222.25 72.39 0)
-			(effects
-				(font
-					(size 1.27 1.27)
-				)
-				(hide yes)
-			)
-		)
-		(property "Description" ""
-			(at 222.25 72.39 0)
-			(effects
-				(font
-					(size 1.27 1.27)
-				)
-				(hide yes)
-			)
-		)
-		(property "PARTREV" "A"
-			(at 222.25 72.39 0)
-			(effects
-				(font
-					(size 1.27 1.27)
-				)
-				(justify bottom)
-				(hide yes)
-			)
-		)
-		(property "STANDARD" "Manufacturer Recommendations"
-			(at 222.25 72.39 0)
-			(effects
-				(font
-					(size 1.27 1.27)
-				)
-				(justify bottom)
-				(hide yes)
-			)
-		)
-		(property "MAXIMUM_PACKAGE_HEIGHT" "2.00 mm"
-			(at 222.25 72.39 0)
-			(effects
-				(font
-					(size 1.27 1.27)
-				)
-				(justify bottom)
-				(hide yes)
-			)
-		)
-		(property "MANUFACTURER" "GCT"
-			(at 222.25 72.39 0)
-			(effects
-				(font
-					(size 1.27 1.27)
-				)
-				(justify bottom)
-				(hide yes)
-			)
-		)
-		(pin "23"
-		)
-		(pin "28"
-		)
-		(pin "S2"
-		)
-		(pin "17"
-		)
-		(pin "36"
-		)
-		(pin "29"
-		)
-		(pin "24"
-		)
-		(pin "20"
-		)
-		(pin "37"
-		)
-		(pin "18"
-		)
-		(pin "35"
-		)
-		(pin "3"
-		)
-		(pin "34"
-		)
-		(pin "6"
-		)
-		(pin "21"
-		)
-		(pin "30"
-		)
-		(pin "13"
-		)
-		(pin "14"
-		)
-		(pin "15"
-		)
-		(pin "25"
-		)
-		(pin "S1"
-		)
-		(pin "22"
-		)
-		(pin "10"
-		)
-		(pin "1"
-		)
-		(pin "11"
-		)
-		(pin "26"
-		)
-		(pin "12"
-		)
-		(pin "31"
-		)
-		(pin "19"
-		)
-		(pin "2"
-		)
-		(pin "16"
-		)
-		(pin "33"
-		)
-		(pin "38"
-		)
-		(pin "39"
-		)
-		(pin "7"
-		)
-		(pin "8"
-		)
-		(pin "4"
-		)
-		(pin "40"
-		)
-		(pin "5"
-		)
-		(pin "9"
-		)
-		(pin "32"
-		)
-		(pin "27"
 		)
 		(instances
 			(project "base"
 				(path "/0b92ad0b-9d78-48b8-8c77-5cb058beae24"
-					(reference "J2")
-					(unit 1)
+					(page "2")
 				)
 			)
